Commit message: Added additional urdfs

File: robots/robot-ee.urdf (robot description, URDF)
Before this commit: robot onshape, 6 links, 5 joints
Links:
- added link end_effector
Joints:
- added joint ee_joint: type revolute, parent wrist_carriage_3, child end_effector, origin xyz=-0.04 0 -0.0485 rpy=0 -1.570796326794896558 0, axis 0 0 1, limit lower=0 upper=6.28318530718 effort=1 velocity=1

Commit message: added physical robot dimensions model

File: robots/robot-ee.urdf (robot description, URDF)
Before this commit: robot onshape, 7 links, 6 joints
Joints:
- joint ee_joint: limit lower=0 upper=6.28318530718 effort=1 velocity=1 -> lower=-3.14159265359 upper=3.14159265359 effort=1 velocity=1
- joint shoulder_bend: limit lower=0 upper=6.28318530718 effort=1 velocity=1 -> lower=-3.14159265359 upper=3.14159265359 effort=1 velocity=1
- joint shoulder_lift: limit lower=0 upper=6.28318530718 effort=1 velocity=1 -> lower=-3.14159265359 upper=3.14159265359 effort=1 velocity=1
- joint shoulder_rotate: limit lower=0 upper=6.28318530718 effort=1 velocity=1 -> lower=-0.52359877559 upper=0.52359877559 effort=1 velocity=1
- joint wrist_1: limit lower=0 upper=6.28318530718 effort=1 velocity=1 -> lower=-3.14159265359 upper=3.14159265359 effort=1 velocity=1
- joint wrist_2: limit lower=0 upper=6.28318530718 effort=1 velocity=1 -> lower=-3.14159265359 upper=3.14159265359 effort=1 velocity=1
